Commit message: aruco

File: src/rosbot_description/urdf/rosbot.xacro (robot description, xacro)
@@ -236,10 +236,21 @@
   </transmission>
   <!-- Orbbec Astra RGBD Camera -->
-  <joint name="astra_joint" type="fixed">
-    <axis xyz="0 0 0" />
+  <joint name="astra_joint" type="continuous">
+    <axis xyz="0 0 1" />
     <origin xyz="-0.03 0 0.18" rpy="0 0 0"/>
     <parent link="body_link"/>
     <child link="camera_link"/>
-  </joint>
+    <limit effort="1" velocity="10"/>
+    <joint_properties damping="5.0" friction="1.0"/>
+  </joint>
+  <transmission name="astra_joint_trans" type="SimpleTransmission">
+    <type>transmission_interface/SimpleTransmission</type>
+    <actuator name="astra_joint_motor">
+      <mechanicalReduction>1</mechanicalReduction>
+    </actuator>
+    <joint name="astra_joint">
+      <hardwareInterface>hardware_interface/EffortJointInterface</hardwareInterface>
+    </joint>
+  </transmission>
   <link name="camera_link">
     <collision>

Commit message: telecamera che gira

File: src/rosbot_description/urdf/rosbot.xacro (robot description, xacro)
@@ -246,11 +246,11 @@
   <transmission name="astra_joint_trans">
     <type>transmission_interface/SimpleTransmission</type>
+    <joint name="astra_joint">
+      <hardwareInterface>hardware_interface/EffortJointInterface</hardwareInterface>
+    </joint>
     <actuator name="astra_joint_motor">
-      <!-- <hardwareInterface>hardware_interface/EffortJointInterface</hardwareInterface> -->
-      <mechanicalReduction>1</mechanicalReduction>
-    </actuator>
-    <joint name="astra_joint">
-      <hardwareInterface>hardware_interface/EffortJointInterface</hardwareInterface>
-    </joint>
+      <hardwareInterface>hardware_interface/EffortJointInterface</hardwareInterface>
+      <mechanicalReduction>1</mechanicalReduction>
+    </actuator>
   </transmission>
   <link name="camera_link">
